Commit message: [Task 2.02]: Integrated gripper into the UR Arm

File: src/my_robot/ur_description/urdf/ur_test_2.urdf.xacro (robot description, xacro)
@@ -4,5 +4,5 @@
    <xacro:arg name="name" default="ur"/>
    <!-- import main macro -->
-   <xacro:include filename="$(find ur_description)/urdf/ur_macro.xacro"/>
+   <xacro:include filename="$(find ur_description)/urdf/ur_macro_2.xacro"/>
    <xacro:include filename="$(find robotnik_sensors)/urdf/all_sensors.urdf.xacro" />
    <!-- possible 'ur_type' values: ur3, ur3e, ur5, ur5e, ur10, ur10e, ur16e, ur20, ur30 -->

File: src/my_robot/ur_description/urdf/ur_test_3.urdf.xacro (robot description, xacro)
@@ -1,14 +1,15 @@
 <?xml version="1.0"?>
-<robot xmlns:xacro="http://wiki.ros.org/xacro" name="$(arg name)">
+<robot xmlns:xacro="http://wiki.ros.org/xacro" name="ur">
    <!-- robot name parameter -->
    <xacro:arg name="name" default="ur"/>
    <!-- import main macro -->
    <xacro:include filename="$(find ur_description)/urdf/ur_macro.xacro"/>
+   <!-- <xacro:include filename="$(find ur_description)/urdf/ur_macro_2.xacro"/> -->
    <xacro:include filename="$(find robotnik_sensors)/urdf/all_sensors.urdf.xacro" />
    <!-- possible 'ur_type' values: ur3, ur3e, ur5, ur5e, ur10, ur10e, ur16e, ur20, ur30 -->
    <!-- the default value should raise an error in case this was called without defining the type -->
-   <xacro:arg name="ur_type" default="ur5x"/>
+   <xacro:arg name="ur_type" default="ur5e"/>
    <!-- parameters -->
-   <xacro:arg name="tf_prefix" default="" />
+   <xacro:arg name="tf_prefix" default="ur5e_" />
    <xacro:arg name="joint_limit_params" default="$(find ur_description)/config/$(arg ur_type)/joint_limits.yaml"/>
    <xacro:arg name="kinematics_params" default="$(find ur_description)/config/$(arg ur_type)/default_kinematics.yaml"/>
@@ -117,5 +118,4 @@
      >
      <origin xyz="0 0 0" rpy="0 0 0" />          <!-- position robot in the world -->
-   </xacro:ur_robot>
 <!-- Vision sensor for color and depth stream of the environment -->
   <xacro:sensor_r430 prefix="top_rgbd" parent="base_link" >
@@ -123,4 +123,6 @@
        <origin xyz="0.6 0.0 1.2" rpy="0 ${pi/2} ${0}"/>
    </xacro:sensor_r430>
+   <!-- </xacro:ur_robot>
+   <xacro:include filename="$(find ur_description)/urdf/gripper.urdf.xacro" /> -->
    <xacro:if value="$(arg sim_gazebo)">
     <!-- Gazebo plugins -->

File: src/my_robot/ur_description/urdf/ur_test_4.urdf.xacro (robot description, xacro)
@@ -1,4 +1,4 @@
 <?xml version="1.0"?>
-<robot xmlns:xacro="http://wiki.ros.org/xacro" name="$(arg name)">
+<robot xmlns:xacro="http://wiki.ros.org/xacro" name="ur">
    <!-- robot name parameter -->
    <xacro:arg name="name" default="ur"/>
@@ -8,5 +8,5 @@
    <!-- possible 'ur_type' values: ur3, ur3e, ur5, ur5e, ur10, ur10e, ur16e, ur20, ur30 -->
    <!-- the default value should raise an error in case this was called without defining the type -->
-   <xacro:arg name="ur_type" default="ur5x"/>
+   <xacro:arg name="ur_type" default="ur5e"/>
    <!-- parameters -->
    <xacro:arg name="tf_prefix" default="" />
@@ -118,7 +118,8 @@
      <origin xyz="0 0 0" rpy="0 0 0" />          <!-- position robot in the world -->
    </xacro:ur_robot>
+  <xacro:include filename="$(find ur_description)/urdf/gripper.urdf.xacro" />
 <!-- Vision sensor for color and depth stream of the environment -->
   <xacro:sensor_r430 prefix="top_rgbd" parent="base_link" >
-       <!--<origin xyz="0.35 0.45 0.1" rpy="0 ${pi/6} ${-pi/2}"/>-->
+             <!-- unused <origin xyz="0.35 0.45 0.1" rpy="0 ${pi/6} ${-pi/2}"/> -->
        <origin xyz="0.6 0.0 1.2" rpy="0 ${pi/2} ${0}"/>
    </xacro:sensor_r430>
