Commit message: [Task 1.03]: Removed extra packages

File: src/my_robot/ur_description/urdf/gripper.urdf.xacro (robot description, xacro)
@@ -242,5 +242,4 @@
             <child link="${prefix}robotiq_85_left_finger_link" />
             <origin xyz="0.03152616 0.0 -0.00376347" rpy="0 0 0" />
-            <!-- <mimic joint="${prefix}robotiq_85_left_knuckle_joint" multiplier="1"/> -->
         </joint>
         <joint name="${prefix}robotiq_85_right_finger_joint" type="fixed">
@@ -248,5 +247,4 @@
             <child link="${prefix}robotiq_85_right_finger_link" />
             <origin xyz="-0.03152616 0.0 -0.00376347" rpy="0 0 0" />
-            <!-- <mimic joint="${prefix}robotiq_85_left_knuckle_joint" multiplier="-1"/> -->
         </joint>
         <joint name="${prefix}robotiq_85_left_inner_knuckle_joint" type="continuous">
@@ -315,5 +313,5 @@
 		        <plugin>gazebo_ros2_control/GazeboSystem</plugin>
 	    	</hardware>
-	    	<joint name="robotiq_85_left_knuckle_joint">
+	    	<joint name="${prefix}robotiq_85_left_knuckle_joint">
 	    		<command_interface name="position">
 	    			<param name="min">0</param>
@@ -333,5 +331,5 @@
     </xacro:if>
     <xacro:if value="${not gripper_only}">
-    	<xacro:robotiq_gripper name="RobotiqGripperHardwareInterface" prefix="" parent="ur5e_tool0" use_fake_hardware="$(arg use_fake_hardware)">
+    	<xacro:robotiq_gripper name="RobotiqGripperHardwareInterface" prefix="" parent="wrist_3_link" use_fake_hardware="$(arg use_fake_hardware)">
         	<origin xyz="0 0 0" rpy="0 0 0" />
     	</xacro:robotiq_gripper>
